File: Weapons/Support/AC-8_Autocannon/Gun/ControlBoard/ControlBoard.kicad_pcb (KiCad board)
At the start: 2 copper layers, 11 parts, among them J1 Conn_01x02, J2 Conn_01x02, J3 TMC_2209_A, J4 TMC_2209_B, J5 Pololu D24V5F5 5V, J6 NEMA-17, J7 NEMA-8, J8 Conn_01x02, J9 Controller_Enable_Switch, U1 Adafruit_QT_Py_RP2040

Commit message: Autocannon Updates
Parts:
- added J10: Conn_01x01, MountingHole:MountingHole_3.2mm_M3, F.Cu at (100.1, 82.3)
- J1, J2, J9: footprint Connector_JST:JST_EH_B2B-EH-A_1x02_P2.50mm_Vertical -> Connector_JST:JST_PH_B2B-PH-K_1x02_P2.00mm_Vertical
- moved J9 98.5 mm to (132.7, 85.7), turned to 90 degrees
- moved J1 94.2 mm to (137.7, 85.7), turned to 90 degrees
- moved J2 82.9 mm to (105.7, 87.4), turned to 180 degrees
- moved J5 65.3 mm to (120.7, 108.0)
- moved D1 63.5 mm to (130.8, 108.0)
- moved J7 20.9 mm to (98.2, 96.5), turned to 0 degrees
- moved J3 13.0 mm to (143.8, 100.2)
- moved J6 12.2 mm to (153.2, 104.0)
- moved J8 8.80 mm to (147.3, 86.4)
- moved U1 6.36 mm to (125.7, 99.9)
- moved J4 1.20 mm to (107.6, 100.2), turned to 180 degrees
Connections:
- U1 pad 1: EN -> DIAG_B
- U1 pad 10: TRIG -> STEP_A
- U1 pad 11: RLOAD -> DIR_A
- U1 pad 3: DIAG_B -> TRIG
- U1 pad 4: DIR_B -> EN
- U1 pad 5: DIR_A -> DIR_B
- U1 pad 6: STEP_A -> STEP_B
- U1 pad 9: STEP_B -> RLOAD
Routing:
- net +24V: track 0.00 -> 88.9 mm
- net +3V3: track 0.00 -> 56.8 mm, vias 0 -> 1
- net EN: track 0.00 -> 46.8 mm, vias 0 -> 2
- net mC-EN: track 0.00 -> 42.6 mm
- net TRIG: track 0.00 -> 26.9 mm, vias 0 -> 1
- net UART_A: track 0.00 -> 26.5 mm, vias 0 -> 1
- net RLOAD: track 0.00 -> 24.9 mm, vias 0 -> 1
- net STEP_A: track 0.00 -> 19.5 mm, vias 0 -> 1
- net DIR_A: track 0.00 -> 17.2 mm
- net GND: track 0.00 -> 15.2 mm, vias 0 -> 19
- net DIR_B: track 0.00 -> 12.4 mm
- net DIAG_B: track 0.00 -> 10.3 mm
- net DIAG_A: track 0.00 -> 10.2 mm
- net UART_B: track 0.00 -> 9.47 mm
- net STEP_B: track 0.00 -> 4.61 mm
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- added copper zone on B.Cu, net +24V
- added copper zone on B.Cu, net GND
- added copper zone on F.Cu, net GND
Other:
- board outline added: 58.4 x 31.8 mm
