File: Weapons/Support/AC-8_Autocannon/Gun/ControlBoard/ControlBoard.kicad_sch (KiCad schematic)
At the start: 11 parts, among them J1 Conn_01x02, J2 Conn_01x02, J3 TMC_2209_A, J4 TMC_2209_B, J5 Pololu D24V5F5 5V, J6 NEMA-17, J7 NEMA-8, J8 Conn_01x02, J9 Controller_Enable_Switch, U1 Adafruit_QT_Py_RP2040

Commit message: Autocannon Updates
Parts:
- added J10: Conn_01x01, MountingHole:MountingHole_3.2mm_M3, symbol Connector_Generic:Conn_01x01
- J1, J2, J9: footprint Connector_JST:JST_EH_B2B-EH-A_1x02_P2.50mm_Vertical -> Connector_JST:JST_PH_B2B-PH-K_1x02_P2.00mm_Vertical
Connections:
- net DIAG_B: now also U1.1 (A0/D0); no longer U1.3 (A2/D2)
- net DIR_A: now also U1.11 (MO/A10/D10); no longer U1.5 (SDA/D4)
- net DIR_B: now also U1.5 (SDA/D4); no longer U1.4 (A3/D3)
- net EN: now also U1.4 (A3/D3); no longer U1.1 (A0/D0)
- net GND: now also J10.1 (Pin_1)
- net RLOAD: now also U1.9 (SCK/A8/D8); no longer U1.11 (MO/A10/D10)
- net STEP_A: now also U1.10 (MI/A9/D9); no longer U1.6 (SCL/D5)
- net STEP_B: now also U1.6 (SCL/D5); no longer U1.9 (SCK/A8/D8)
- net TRIG: now also U1.3 (A2/D2); no longer U1.10 (MI/A9/D9)
Changed lines of the file:
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@@
+    (stroke (width 0) (type default) (color 0 0 0 0))
+  )
+  (wire (pts (xy 94.615 126.365) (xy 94.615 156.21))
     (stroke (width 0) (type default) (color 0 0 0 0))
   )
@@
     (stroke (width 0) (type default) (color 0 0 0 0))
   )
+  (wire (pts (xy 92.71 126.365) (xy 94.615 126.365))
+    (stroke (width 0) (type default) (color 0 0 0 0))
+  )
   (wire (pts (xy 151.765 60.325) (xy 151.765 62.23))
     (stroke (width 0) (type default) (color 0 0 0 0))
@@
     )
   )
-  (global_label "DIR_B" (shape input) (at 46.99 50.165 180) (fields_autoplaced)
-    (effects (font (size 1.27 1.27)) (justify right))
-    (property "Intersheet References" "${INTERSHEET_REFS}" (id 0) (at 39.1945 50.0856 0)
+  (global_label "DIR_B" (shape input) (at 46.99 52.705 180) (fields_autoplaced)
+    (effects (font (size 1.27 1.27)) (justify right))
+    (property "Intersheet References" "${INTERSHEET_REFS}" (id 0) (at 39.1945 52.6256 0)
       (effects (font (size 1.27 1.27)) (justify right) hide)
     )
@@
     )
   )
-  (global_label "DIR_A" (shape input) (at 46.99 52.705 180) (fields_autoplaced)
-    (effects (font (size 1.27 1.27)) (justify right))
-    (property "Intersheet References" "${INTERSHEET_REFS}" (id 0) (at 39.3759 52.6256 0)
-      (effects (font (size 1.27 1.27)) (justify right) hide)
+  (global_label "DIR_A" (shape input) (at 80.01 50.165 0) (fields_autoplaced)
+    (effects (font (size 1.27 1.27)) (justify left))
+    (property "Intersheet References" "${INTERSHEET_REFS}" (id 0) (at 87.6241 50.2444 0)
+      (effects (font (size 1.27 1.27)) (justify left) hide)
     )
   )
@@
     )
   )
-  (global_label "EN" (shape input) (at 46.99 42.545 180) (fields_autoplaced)
-    (effects (font (size 1.27 1.27)) (justify right))
-    (property "Intersheet References" "${INTERSHEET_REFS}" (id 0) (at 42.0974 42.4656 0)
+  (global_label "EN" (shape input) (at 46.99 50.165 180) (fields_autoplaced)
+    (effects (font (size 1.27 1.27)) (justify right))
+    (property "Intersheet References" "${INTERSHEET_REFS}" (id 0) (at 42.0974 50.0856 0)
       (effects (font (size 1.27 1.27)) (justify right) hide)
     )
@@
     )
   )
-  (global_label "DIAG_B" (shape input) (at 46.99 47.625 180) (fields_autoplaced)
-    (effects (font (size 1.27 1.27)) (justify right))
-    (property "Intersheet References" "${INTERSHEET_REFS}" (id 0) (at 38.1059 47.5456 0)
-      (effects (font (size 1.27 1.27)) (justify right) hide)
-    )
-  )
-  (global_label "STEP_A" (shape input) (at 46.99 55.245 180) (fields_autoplaced)
-    (effects (font (size 1.27 1.27)) (justify right))
-    (property "Intersheet References" "${INTERSHEET_REFS}" (id 0) (at 37.9245 55.1656 0)
-      (effects (font (size 1.27 1.27)) (justify right) hide)
+  (global_label "DIAG_B" (shape input) (at 46.99 42.545 180) (fields_autoplaced)
+    (effects (font (size 1.27 1.27)) (justify right))
+    (property "Intersheet References" "${INTERSHEET_REFS}" (id 0) (at 38.1059 42.4656 0)
+      (effects (font (size 1.27 1.27)) (justify right) hide)
+    )
+  )
+  (global_label "STEP_A" (shape input) (at 80.01 52.705 0) (fields_autoplaced)
+    (effects (font (size 1.27 1.27)) (justify left))
+    (property "Intersheet References" "${INTERSHEET_REFS}" (id 0) (at 89.0755 52.7844 0)
+      (effects (font (size 1.27 1.27)) (justify left) hide)
     )
   )
@@
     )
   )
-  (global_label "RLOAD" (shape input) (at 80.01 50.165 0) (fields_autoplaced)
-    (effects (font (size 1.27 1.27)) (justify left))
-    (property "Intersheet References" "${INTERSHEET_REFS}" (id 0) (at 88.4102 50.0856 0)
+  (global_label "RLOAD" (shape input) (at 80.01 55.245 0) (fields_autoplaced)
+    (effects (font (size 1.27 1.27)) (justify left))
+    (property "Intersheet References" "${INTERSHEET_REFS}" (id 0) (at 88.4102 55.1656 0)
       (effects (font (size 1.27 1.27)) (justify left) hide)
     )
@@
     )
   )
-  (global_label "STEP_B" (shape input) (at 80.01 55.245 0) (fields_autoplaced)
-    (effects (font (size 1.27 1.27)) (justify left))
-    (property "Intersheet References" "${INTERSHEET_REFS}" (id 0) (at 89.2569 55.3244 0)
-      (effects (font (size 1.27 1.27)) (justify left) hide)
+  (global_label "STEP_B" (shape input) (at 46.99 55.245 180) (fields_autoplaced)
+    (effects (font (size 1.27 1.27)) (justify right))
+    (property "Intersheet References" "${INTERSHEET_REFS}" (id 0) (at 37.7431 55.1656 0)
+      (effects (font (size 1.27 1.27)) (justify right) hide)
     )
   )
@@
     )
   )
-  (global_label "TRIG" (shape input) (at 80.01 52.705 0) (fields_autoplaced)
-    (effects (font (size 1.27 1.27)) (justify left))
-    (property "Intersheet References" "${INTERSHEET_REFS}" (id 0) (at 86.5355 52.6256 0)
-      (effects (font (size 1.27 1.27)) (justify left) hide)
+  (global_label "TRIG" (shape input) (at 46.99 47.625 180) (fields_autoplaced)
+    (effects (font (size 1.27 1.27)) (justify right))
+    (property "Intersheet References" "${INTERSHEET_REFS}" (id 0) (at 40.4645 47.7044 0)
+      (effects (font (size 1.27 1.27)) (justify right) hide)
     )
   )
@@
     )
     (property "Datasheet" "" (id 3) (at 103.505 62.23 0)
+      (effects (font (size 1.27 1.27)) hide)
+    )
+    (pin "1")
+  )
+  (symbol (lib_id "Connector_Generic:Conn_01x01") (at 87.63 126.365 180) (unit 1)
+    (in_bom yes) (on_board yes) (fields_autoplaced)
+    (property "Reference" "J10" (id 0) (at 87.63 121.1285 0))
+    (property "Value" "Conn_01x01" (id 1) (at 87.63 123.9036 0))
+    (property "Footprint" "MountingHole:MountingHole_3.2mm_M3" (id 2) (at 87.63 126.365 0)
+      (effects (font (size 1.27 1.27)) hide)
+    )
+    (property "Datasheet" "~" (id 3) (at 87.63 126.365 0)
       (effects (font (size 1.27 1.27)) hide)
     )
@@
       (effects (font (size 1.27 1.27)) (justify left))
     )
-    (property "Footprint" "Connector_JST:JST_EH_B2B-EH-A_1x02_P2.50mm_Vertical" (id 2) (at 66.675 92.075 0)
+    (property "Footprint" "Connector_JST:JST_PH_B2B-PH-K_1x02_P2.00mm_Vertical" (id 2) (at 66.675 92.075 0)
       (effects (font (size 1.27 1.27)) hide)
     )
@@
     (pin "1")
   )
+  (symbol (lib_id "power:GND") (at 94.615 156.21 0) (unit 1)
+    (in_bom yes) (on_board yes) (fields_autoplaced)
+    (property "Reference" "#PWR0120" (id 0) (at 94.615 162.56 0)
+      (effects (font (size 1.27 1.27)) hide)
+    )
+    (property "Value" "GND" (id 1) (at 94.615 160.7725 0))
+    (property "Footprint" "" (id 2) (at 94.615 156.21 0)
+      (effects (font (size 1.27 1.27)) hide)
+    )
+    (property "Datasheet" "" (id 3) (at 94.615 156.21 0)
+      (effects (font (size 1.27 1.27)) hide)
+    )
+    (pin "1")
+  )
   (symbol (lib_id "Connector_Generic:Conn_01x02") (at 259.715 39.37 0) (mirror y) (unit 1)
     (in_bom yes) (on_board yes) (fields_autoplaced)
     (property "Reference" "J9" (id 0) (at 259.715 34.1335 0))
     (property "Value" "Controller_Enable_Switch" (id 1) (at 259.715 36.9086 0))
-    (property "Footprint" "Connector_JST:JST_EH_B2B-EH-A_1x02_P2.50mm_Vertical" (id 2) (at 259.715 39.37 0)
+    (property "Footprint" "Connector_JST:JST_PH_B2B-PH-K_1x02_P2.00mm_Vertical" (id 2) (at 259.715 39.37 0)
       (effects (font (size 1.27 1.27)) hide)
     )
@@
       (effects (font (size 1.27 1.27)) (justify left))
     )
-    (property "Footprint" "Connector_JST:JST_EH_B2B-EH-A_1x02_P2.50mm_Vertical" (id 2) (at 66.675 80.01 0)
+    (property "Footprint" "Connector_JST:JST_PH_B2B-PH-K_1x02_P2.00mm_Vertical" (id 2) (at 66.675 80.01 0)
       (effects (font (size 1.27 1.27)) hide)
     )
@@
       (reference "#PWR0119") (unit 1) (value "GND") (footprint "")
     )
+    (path "/80fe070c-5552-4d5b-9daf-e06941e95f16"
+      (reference "#PWR0120") (unit 1) (value "GND") (footprint "")
+    )
     (path "/16943b7c-09b7-48ab-9c63-c72f1d3a56d6"
       (reference "D1") (unit 1) (value "D") (footprint "Diode_SMD:D_0603_1608Metric_Pad1.05x0.95mm_HandSolder")
     )
     (path "/94797e3b-979a-44a0-874b-8f12d3eff9f7"
-      (reference "J1") (unit 1) (value "Conn_01x02") (footprint "Connector_JST:JST_EH_B2B-EH-A_1x02_P2.50mm_Vertical")
+      (reference "J1") (unit 1) (value "Conn_01x02") (footprint "Connector_JST:JST_PH_B2B-PH-K_1x02_P2.00mm_Vertical")
     )
     (path "/3fdf4732-4e13-4fab-b87a-b5c440a32e5b"
-      (reference "J2") (unit 1) (value "Conn_01x02") (footprint "Connector_JST:JST_EH_B2B-EH-A_1x02_P2.50mm_Vertical")
+      (reference "J2") (unit 1) (value "Conn_01x02") (footprint "Connector_JST:JST_PH_B2B-PH-K_1x02_P2.00mm_Vertical")
     )
     (path "/b2b89835-e5fd-4978-acd2-b15f779fa069"
@@
     )
     (path "/8901b55f-ec61-44e5-a9db-df3fda309f28"
-      (reference "J9") (unit 1) (value "Controller_Enable_Switch") (footprint "Connector_JST:JST_EH_B2B-EH-A_1x02_P2.50mm_Vertical")
+      (reference "J9") (unit 1) (value "Controller_Enable_Switch") (footprint "Connector_JST:JST_PH_B2B-PH-K_1x02_P2.00mm_Vertical")
+    )
+    (path "/1560abd3-82b8-47b3-8a71-c7983ddb54c7"
+      (reference "J10") (unit 1) (value "Conn_01x01") (footprint "MountingHole:MountingHole_3.2mm_M3")
     )
     (path "/2a468805-02e1-42b1-ade3-6a84063ab293"
